File: hardware/schematics/address_logic/address_logic.sch (KiCad schematic (older format))
At the start: 27 parts

Commit message: I started working on the PCBs
Parts:
- added C1, C2, C3, C4, C5, C6, C7, C8: 0.1uF, Capacitor_THT:C_Disc_D3.8mm_W2.6mm_P2.50mm, symbol Device:C
- added unit 3 of U1
- added unit 5 of U2
- added unit 5 of U3
- added unit 7 of U4
- added unit 5 of U5
- added unit 3 of U6
- added unit 7 of U7
- added unit 5 of U8
- J1: renamed from J?; footprint (none) -> m6502:PinHeader_2x20_P2.54mm_Horizontal_Counter_Clockwise
- U1, U2, U3, U4, U5, U6, U7, U8: renamed from U?; footprint (none) -> Package_DIP:DIP-14_W7.62mm_Socket
Connections:
- net A0: no longer J1.3 (Pin_3)
- net A1: no longer J1.4 (Pin_4)
- net GND: now also C1.2, C2.2, C3.2, C4.2, C5.2, C6.2, C7.2, C8.2, U1.7 (GND), U2.7 (GND), U3.7 (GND), U4.7 (GND), U5.7 (GND), U6.7 (GND), U7.7 (GND), U8.7 (GND)
- net RESET: no longer J1.2 (Pin_2)
- net ROM renamed A15
- net VCC renamed +5V
- net +5V: now also C1.1, C2.1, C3.1, C4.1, C5.1, C6.1, C7.1, C8.1, U1.14 (VCC), U2.14 (VCC), U3.14 (VCC), U4.14 (VCC), U5.14 (VCC), U6.14 (VCC), U7.14 (VCC), U8.14 (VCC)
- no-connect marks 0 -> 16
Other:
- moved on the sheet: U7C, U7D, U8C, U8D
